File: KiCad/Fernschreiber.sch (KiCad schematic (older format))
At the start: 30 parts, among them J1 Teleprinter, J10 Test_Conn_write, J11 Test_Conn_Lesen_b_opto, J2 Step-Up, J3 18,19,23,3V3,GND, J4 12,13,14,3V3,GND, J5 TX,RX,3V3,GND, J6 5V, J7 Test_Conn_3V3, J8 Test_Conn_Voltage_reversal, J9 Test_Conn_read, K1 FINDER-40.41, K2 FINDER-40.41, Q1 Q_NMOS_SGD, Q2 Q_NMOS_SGD, U1 4N28, U2 ESP32_Joy-it, U3 4N28

Commit message: Updated PCB
Parts:
- added C1, C2, C3: CAP, Capacitor_THT:CP_Radial_D8.0mm_P3.50mm, symbol pspice:CAP
- added H1, H2, H3, H4: MountingHole_Pad, Fernschreiber:Hole, symbol Mechanical:MountingHole_Pad
- added J12: Conn_01x05_Male, Fernschreiber:stepdown, symbol Connector:Conn_01x05_Male
Connections:
- net 5V: now also C1.1, C2.1, C3.1, J12.1 (Pin_1); no longer J6.2 (Pin_2)
- net GND: now also C1.2, C2.2, C3.2, H1.1, H2.1, H3.1, H4.1, J12.3 (Pin_3), J12.4 (Pin_4), J12.5 (Pin_5)
- new net 5V_12V: J12.2 (Pin_2), J6.2 (Pin_2)
Other:
- moved on the sheet: J6
Changed lines of the file:
@@
 L Connector:Conn_01x02_Female J6
 U 1 1 6051B127
-P 6050 3250
-F 0 "J6" V 5988 3062 50  0000 R CNN
-F 1 "5V" V 5897 3062 50  0000 R CNN
-F 2 "Fernschreiber:DECA MB310-500M02 Schraubklemmblock" H 6050 3250 50  0001 C CNN
-F 3 "~" H 6050 3250 50  0001 C CNN
-	1    6050 3250
-	0    -1   -1   0
-$EndComp
-Text Label 6150 3600 0    50   ~ 0
-5V
-Wire Wire Line
-	6150 3450 6150 3600
+P 6600 3300
+F 0 "J6" V 6538 3112 50  0000 R CNN
+F 1 "5V" V 6447 3112 50  0000 R CNN
+F 2 "Fernschreiber:DECA MB310-500M02 Schraubklemmblock" H 6600 3300 50  0001 C CNN
+F 3 "~" H 6600 3300 50  0001 C CNN
+	1    6600 3300
+	0    -1   -1   0
+$EndComp
+Text Label 6700 3650 0    50   ~ 0
+5V_12V
+Wire Wire Line
+	6700 3500 6700 3650
 Text Label 1300 1200 2    50   ~ 0
 5V
@@
 L power:GND #PWR05
 U 1 1 60537F40
-P 6050 3500
-F 0 "#PWR05" H 6050 3250 50  0001 C CNN
-F 1 "GND" H 6055 3327 50  0000 C CNN
-F 2 "" H 6050 3500 50  0001 C CNN
-F 3 "" H 6050 3500 50  0001 C CNN
-	1    6050 3500
-	1    0    0    -1
-$EndComp
-Wire Wire Line
-	6050 3450 6050 3500
+P 6600 3550
+F 0 "#PWR05" H 6600 3300 50  0001 C CNN
+F 1 "GND" H 6605 3377 50  0000 C CNN
+F 2 "" H 6600 3550 50  0001 C CNN
+F 3 "" H 6600 3550 50  0001 C CNN
+	1    6600 3550
+	1    0    0    -1
+$EndComp
+Wire Wire Line
+	6600 3500 6600 3550
 Wire Wire Line
 	7500 3300 7500 3500
@@
 	5900 500  5900 3000
 Wire Notes Line
-	4000 5000 500  5000
-Wire Notes Line
 	4000 4000 8000 4000
 Text Label 8900 2500 2    50   ~ 0
@@
 Wire Wire Line
 	8900 2500 8950 2500
+$Comp
+L pspice:CAP C1
+U 1 1 6047BBD7
+P 4550 4450
+F 0 "C1" H 4728 4496 50  0000 L CNN
+F 1 "CAP" H 4728 4405 50  0000 L CNN
+F 2 "Capacitor_THT:CP_Radial_D8.0mm_P3.50mm" H 4550 4450 50  0001 C CNN
+F 3 "~" H 4550 4450 50  0001 C CNN
+	1    4550 4450
+	1    0    0    -1
+$EndComp
+$Comp
+L pspice:CAP C2
+U 1 1 60480AB7
+P 5800 4450
+F 0 "C2" H 5978 4496 50  0000 L CNN
+F 1 "CAP" H 5978 4405 50  0000 L CNN
+F 2 "Capacitor_THT:CP_Radial_D8.0mm_P3.50mm" H 5800 4450 50  0001 C CNN
+F 3 "~" H 5800 4450 50  0001 C CNN
+	1    5800 4450
+	1    0    0    -1
+$EndComp
+$Comp
+L pspice:CAP C3
+U 1 1 60483B5B
+P 7050 4450
+F 0 "C3" H 7228 4496 50  0000 L CNN
+F 1 "CAP" H 7228 4405 50  0000 L CNN
+F 2 "Capacitor_THT:CP_Radial_D8.0mm_P3.50mm" H 7050 4450 50  0001 C CNN
+F 3 "~" H 7050 4450 50  0001 C CNN
+	1    7050 4450
+	1    0    0    -1
+$EndComp
+Text Label 7050 4200 0    50   ~ 0
+5V
+Text Label 5800 4200 0    50   ~ 0
+5V
+Text Label 4550 4200 0    50   ~ 0
+5V
+$Comp
+L power:GND #PWR0101
+U 1 1 60492586
+P 4550 4700
+F 0 "#PWR0101" H 4550 4450 50  0001 C CNN
+F 1 "GND" H 4555 4527 50  0000 C CNN
+F 2 "" H 4550 4700 50  0001 C CNN
+F 3 "" H 4550 4700 50  0001 C CNN
+	1    4550 4700
+	1    0    0    -1
+$EndComp
+$Comp
+L power:GND #PWR0102
+U 1 1 604951FB
+P 5800 4700
+F 0 "#PWR0102" H 5800 4450 50  0001 C CNN
+F 1 "GND" H 5805 4527 50  0000 C CNN
+F 2 "" H 5800 4700 50  0001 C CNN
+F 3 "" H 5800 4700 50  0001 C CNN
+	1    5800 4700
+	1    0    0    -1
+$EndComp
+$Comp
+L power:GND #PWR0103
+U 1 1 60498193
+P 7050 4700
+F 0 "#PWR0103" H 7050 4450 50  0001 C CNN
+F 1 "GND" H 7055 4527 50  0000 C CNN
+F 2 "" H 7050 4700 50  0001 C CNN
+F 3 "" H 7050 4700 50  0001 C CNN
+	1    7050 4700
+	1    0    0    -1
+$EndComp
+Wire Notes Line
+	500  5000 8000 5000
+Text Label 5650 3300 0    50   ~ 0
+5V
+Text Label 5650 3400 0    50   ~ 0
+5V_12V
+$Comp
+L Connector:Conn_01x05_Male J12
+U 1 1 604EC90B
+P 5300 3500
+F 0 "J12" H 5408 3881 50  0000 C CNN
+F 1 "Conn_01x05_Male" H 5408 3790 50  0000 C CNN
+F 2 "Fernschreiber:stepdown" H 5300 3500 50  0001 C CNN
+F 3 "~" H 5300 3500 50  0001 C CNN
+	1    5300 3500
+	1    0    0    -1
+$EndComp
+$Comp
+L power:GND #PWR0104
+U 1 1 60500A2C
+P 5650 3700
+F 0 "#PWR0104" H 5650 3450 50  0001 C CNN
+F 1 "GND" H 5655 3527 50  0000 C CNN
+F 2 "" H 5650 3700 50  0001 C CNN
+F 3 "" H 5650 3700 50  0001 C CNN
+	1    5650 3700
+	1    0    0    -1
+$EndComp
+Wire Wire Line
+	5500 3500 5650 3500
+Wire Wire Line
+	5650 3500 5650 3600
+Wire Wire Line
+	5500 3600 5650 3600
+Connection ~ 5650 3600
+Wire Wire Line
+	5650 3600 5650 3700
+Wire Wire Line
+	5500 3700 5650 3700
+Connection ~ 5650 3700
+Wire Wire Line
+	5500 3400 5650 3400
+Wire Wire Line
+	5500 3300 5650 3300
+$Comp
+L Mechanical:MountingHole_Pad H2
+U 1 1 604C43A9
+P 4350 5500
+F 0 "H2" V 4587 5503 50  0000 C CNN
+F 1 "MountingHole_Pad" V 4496 5503 50  0000 C CNN
+F 2 "Fernschreiber:Hole" H 4350 5500 50  0001 C CNN
+F 3 "~" H 4350 5500 50  0001 C CNN
+	1    4350 5500
+	0    -1   -1   0
+$EndComp
+$Comp
+L Mechanical:MountingHole_Pad H3
+U 1 1 604C9F4C
+P 4350 5750
+F 0 "H3" V 4587 5753 50  0000 C CNN
+F 1 "MountingHole_Pad" V 4496 5753 50  0000 C CNN
+F 2 "Fernschreiber:Hole" H 4350 5750 50  0001 C CNN
+F 3 "~" H 4350 5750 50  0001 C CNN
+	1    4350 5750
+	0    -1   -1   0
+$EndComp
+$Comp
+L Mechanical:MountingHole_Pad H4
+U 1 1 604CD357
+P 4350 6000
+F 0 "H4" V 4587 6003 50  0000 C CNN
+F 1 "MountingHole_Pad" V 4496 6003 50  0000 C CNN
+F 2 "Fernschreiber:Hole" H 4350 6000 50  0001 C CNN
+F 3 "~" H 4350 6000 50  0001 C CNN
+	1    4350 6000
+	0    -1   -1   0
+$EndComp
+$Comp
+L Mechanical:MountingHole_Pad H1
+U 1 1 604D06A9
+P 4350 5250
+F 0 "H1" V 4587 5253 50  0000 C CNN
+F 1 "MountingHole_Pad" V 4496 5253 50  0000 C CNN
+F 2 "Fernschreiber:Hole" H 4350 5250 50  0001 C CNN
+F 3 "~" H 4350 5250 50  0001 C CNN
+	1    4350 5250
+	0    -1   -1   0
+$EndComp
+$Comp
+L power:GND #PWR0105
+U 1 1 604E2513
+P 4450 6050
+F 0 "#PWR0105" H 4450 5800 50  0001 C CNN
+F 1 "GND" H 4455 5877 50  0000 C CNN
+F 2 "" H 4450 6050 50  0001 C CNN
+F 3 "" H 4450 6050 50  0001 C CNN
+	1    4450 6050
+	1    0    0    -1
+$EndComp
+Wire Wire Line
+	4450 5250 4450 5500
+Wire Wire Line
+	4450 5500 4450 5750
+Connection ~ 4450 5500
+Wire Wire Line
+	4450 5750 4450 6000
+Connection ~ 4450 5750
+Wire Wire Line
+	4450 6000 4450 6050
+Connection ~ 4450 6000
 $EndSCHEMATC
