File: KiCad/Fernschreiber.kicad_pcb (KiCad board)
At the start: 2 copper layers, 39 parts, among them J1 Test_Conn_Spannungsumkehr, J10 TX,RX,3V3,GND, J11 12,13,14,3V3,GND, J12 18,19,23,3V3,GND, J2 Test_Conn_5V, J3 Fernschreiber, J4 Test_Conn_Lesen_b_opto, J5 Step-Up, J6 Test_Conn_3V3, J7 12V, J8 Test_Conn_Lesen_a_opto, J9 Test_Conn_Schreiben, K1 FINDER-40.41, K2 FINDER-40.41, Q1 Q_NMOS_SGD, Q2 Q_NMOS_SGD, U1 4N28, U2 4N28, U3 ESP32-WROOM-32

Commit message: Finished routing PCB + updated Footprints + updated Symbols + updated Schematic + ordered PCB at JLCPCB
Parts:
- added G***: LOGO, Fernschreiber:Signatur, F.Cu at (139.8, 58.4)
- added G***: LOGO, Fernschreiber:HTR_Logo, F.Cu at (125.0, 61.0)
- added REF**: Hole, Fernschreiber:Hole, F.Cu at (61.0, 136.1)
- added REF**: Hole, Fernschreiber:Hole, F.Cu at (51.1, 46.1)
- added REF**: Hole, Fernschreiber:Hole, F.Cu at (141.2, 136.3)
- added REF**: Hole, Fernschreiber:Hole, F.Cu at (141.1, 46.1)
- J10: value TX,RX,3V3,GND -> 18,19,23,3V3,GND; footprint Connector_PinHeader_2.54mm:PinHeader_1x04_P2.54mm_Vertical -> Connector_PinHeader_2.54mm:PinHeader_1x05_P2.54mm_Vertical
- J12: value 18,19,23,3V3,GND -> TX,RX,3V3,GND; footprint Connector_PinHeader_2.54mm:PinHeader_1x05_P2.54mm_Vertical -> Connector_PinHeader_2.54mm:PinHeader_1x04_P2.54mm_Vertical
- J4: value Test_Conn_Lesen_b_opto -> Test_Conn_Schreiben_D17
- J5: value Step-Up -> Test_Conn_Lesen_b_opto; footprint Fernschreiber:DECA MB310-500M02 Schraubklemmblock -> Connector_PinHeader_2.54mm:PinHeader_1x01_P2.54mm_Vertical
- J6: value Test_Conn_3V3 -> Step-Up; footprint Connector_PinHeader_2.54mm:PinHeader_1x02_P2.54mm_Vertical -> Fernschreiber:DECA MB310-500M02 Schraubklemmblock
- J7: value 12V -> Test_Conn_3V3; footprint Fernschreiber:DECA MB310-500M02 Schraubklemmblock -> Connector_PinHeader_2.54mm:PinHeader_1x02_P2.54mm_Vertical
- J8: value Test_Conn_Lesen_a_opto -> Test_Conn_Lesen_a_opto_D16
- J9: value Test_Conn_Schreiben -> 12V; footprint Connector_PinHeader_2.54mm:PinHeader_1x01_P2.54mm_Vertical -> Fernschreiber:DECA MB310-500M02 Schraubklemmblock
- U3: value ESP32-WROOM-32 -> ESP32_Joy-it
- moved J4 163.3 mm to (60.8, 128.7)
- moved J8 158.5 mm to (82.8, 108.1)
- moved R2 126.5 mm to (111.1, 102.5), turned to 180 degrees
- moved U1 123.2 mm to (99.2, 83.9), turned to 270 degrees
- moved R1 113.0 mm to (70.0, 91.1)
- moved U3 112.3 mm to (71.8, 64.6), turned to 180 degrees
- moved J2 104.6 mm to (127.4, 99.9), turned to 0 degrees
- moved J1 101.6 mm to (103.0, 76.3)
- moved J7 93.9 mm to (103.0, 68.2)
- moved D4 79.4 mm to (122.3, 113.2)
- moved J6 78.2 mm to (92.1, 136.0), turned to 0 degrees
- moved J3 74.7 mm to (116.0, 136.0), turned to 0 degrees
- moved K2 74.6 mm to (125.9, 121.5), turned to 270 degrees
- moved K1 73.8 mm to (94.6, 121.5), turned to 270 degrees
- moved Q1 72.1 mm to (109.1, 89.3), turned to 270 degrees
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Connections:
- J10 pad 1: GND -> /3V3
- J10 pad 2: /3V3 -> GND
- J10 pad 3: (no net) -> /D18
- J10 pad 4: (no net) -> /D19
- J11 pad 1: GND -> /3V3
- J11 pad 2: /3V3 -> GND
- J11 pad 3: Net-(J11-Pad3) -> /D12
- J11 pad 4: Net-(J11-Pad4) -> /D13
- J11 pad 5: Net-(J11-Pad5) -> /D14
- J12 pad 1: GND -> /3V3
- J12 pad 2: /3V3 -> GND
- J12 pad 3: Net-(J12-Pad3) -> /RX0
- J12 pad 4: (no net) -> /TX0
- J4 pad 1: GND -> Net-(J4-Pad1)
- J5 pad 1: Net-(C3-Pad1) -> Net-(J5-Pad1)
- J6 pad 2: /3V3 -> Net-(C3-Pad1)
- J7 pad 2: +12V -> /3V3
- J8 pad 1: (no net) -> Net-(J8-Pad1)
- J9 pad 1: (no net) -> +12V
- Q2 pad 2: Net-(Q2-Pad2) -> Net-(J4-Pad1)
- R1 pad 1: /Spannungsumkehr -> /Spannungsumkehr_Relai
- R3 pad 1: Net-(Q2-Pad2) -> Net-(J4-Pad1)
- R8 pad 2: Net-(R8-Pad2) -> Net-(J5-Pad1)
- R9 pad 2: Net-(R9-Pad2) -> Net-(J8-Pad1)
- U2 pad 1: Net-(R8-Pad2) -> Net-(J5-Pad1)
- U2 pad 5: Net-(R9-Pad2) -> Net-(J8-Pad1)
Routing:
- net /3V3: track 0.00 -> 196.2 mm
- net Net-(D3-Pad1): track 0.00 -> 100.1 mm
- net Net-(5V1-Pad3): track 0.00 -> 86.7 mm
- net Net-(C3-Pad1): track 0.00 -> 82.7 mm
- net Net-(D1-Pad2): track 0.00 -> 82.5 mm
- net GND: track 0.00 -> 77.0 mm
- net Net-(J4-Pad1): track 0.00 -> 62.5 mm
- net Net-(J8-Pad1): track 0.00 -> 54.1 mm
- net /D23: track 0.00 -> 48.7 mm
- net +12V: track 0.00 -> 43.5 mm
- net /RX0: track 0.00 -> 37.4 mm
- net /TX0: track 0.00 -> 37.4 mm
- net /D19: track 0.00 -> 37.1 mm
- net /D18: track 0.00 -> 32.7 mm
- net Net-(J3-Pad1): track 0.00 -> 30.7 mm
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- added copper zone on B.Cu, net GND
- added copper zone on F.Cu, net GND
Other:
- board outline added: 100 x 100 mm
- board text added: "J1 : Relay Controll J2 : GND 5V J3 : Teleprinter Connetion J4 : Write J5 : Read befor Opto J6 : Step-Up 60V J7 : GND 3V3 J8 : Read after Opto J9 : Supply 12V J10: 3V3 GND D18 D19 D23 J11: 3V3 GND D12 D13 D14 J12: 3V3 GND RX0 TX0"
- board text added: "Power 12V"
- board text added: "Step-Up 60V"
- board text added: "Teleprinter"
- board text added: "Teleprinter-FSG Rev. 1 Design by Metzler Benedikt"

Commit message: Rev.2 PCB
Parts:
- removed 3V1: LD1117, Fernschreiber:LD1117
- removed 5V1: L7805, Fernschreiber:L7805AB
- removed C1, C2, C3, C4, C5: CAP, Capacitor_THT:CP_Radial_D7.5mm_P2.50mm
- removed D4: 1N5711, Diode_THT:D_DO-35_SOD27_P7.62mm_Horizontal
- removed G***: LOGO, Fernschreiber:Signatur
- removed G***: LOGO, Fernschreiber:HTR_Logo
- removed J12: TX,RX,3V3,GND, Connector_PinHeader_2.54mm:PinHeader_1x04_P2.54mm_Vertical
- removed REF** (x4): Hole, Fernschreiber:Hole
- D1, D2, D3: footprint Diode_THT:D_DO-35_SOD27_P7.62mm_Horizontal -> Diode_THT:D_DO-201AE_P15.24mm_Horizontal
- J1: value Test_Conn_Spannungsumkehr -> Teleprinter; footprint Connector_PinHeader_2.54mm:PinHeader_1x01_P2.54mm_Vertical -> Fernschreiber:DECA MB310-500M02 Schraubklemmblock
- J10: value 18,19,23,3V3,GND -> Test_Conn_write; footprint Connector_PinHeader_2.54mm:PinHeader_1x05_P2.54mm_Vertical -> Connector_PinHeader_2.54mm:PinHeader_1x01_P2.54mm_Vertical
- J11: value 12,13,14,3V3,GND -> Test_Conn_Lesen_b_opto; footprint Connector_PinHeader_2.54mm:PinHeader_1x05_P2.54mm_Vertical -> Connector_PinHeader_2.54mm:PinHeader_1x01_P2.54mm_Vertical
- J2: value Test_Conn_5V -> Step-Up; footprint Connector_PinHeader_2.54mm:PinHeader_1x02_P2.54mm_Vertical -> Fernschreiber:DECA MB310-500M02 Schraubklemmblock
- J3: value Fernschreiber -> 18,19,23,3V3,GND; footprint Fernschreiber:DECA MB310-500M02 Schraubklemmblock -> Connector_PinHeader_2.54mm:PinHeader_1x05_P2.54mm_Vertical
- J4: value Test_Conn_Schreiben_D17 -> 12,13,14,3V3,GND; footprint Connector_PinHeader_2.54mm:PinHeader_1x01_P2.54mm_Vertical -> Connector_PinHeader_2.54mm:PinHeader_1x05_P2.54mm_Vertical
- J5: value Test_Conn_Lesen_b_opto -> TX,RX,3V3,GND; footprint Connector_PinHeader_2.54mm:PinHeader_1x01_P2.54mm_Vertical -> Connector_PinHeader_2.54mm:PinHeader_1x04_P2.54mm_Vertical
- J6: value Step-Up -> 5V
- J8: value Test_Conn_Lesen_a_opto_D16 -> Test_Conn_Voltage_reversal
- J9: value 12V -> Test_Conn_read; footprint Fernschreiber:DECA MB310-500M02 Schraubklemmblock -> Connector_PinHeader_2.54mm:PinHeader_1x01_P2.54mm_Vertical
- R1, R2, R9: footprint Resistor_THT:R_Axial_DIN0414_L11.9mm_D4.5mm_P20.32mm_Horizontal -> Resistor_THT:R_Axial_DIN0411_L9.9mm_D3.6mm_P12.70mm_Horizontal
- R3: value 1k -> 3x1k; footprint Resistor_THT:R_Axial_DIN0414_L11.9mm_D4.5mm_P20.32mm_Horizontal -> Fernschreiber:3X1k_Parallel
- R7: value 3x1k -> 1k; footprint Fernschreiber:3X1k_Parallel -> Resistor_THT:R_Axial_DIN0411_L9.9mm_D3.6mm_P12.70mm_Horizontal
- R8: footprint Resistor_THT:R_Axial_DIN0414_L11.9mm_D4.5mm_P25.40mm_Horizontal -> Resistor_THT:R_Axial_DIN0414_L11.9mm_D4.5mm_P15.24mm_Horizontal
- U2: value 4N28 -> ESP32_Joy-it; footprint Fernschreiber:IC-Fassung-6pol -> Fernschreiber:ESP32_Joy-it
- U3: value ESP32_Joy-it -> 4N28; footprint Fernschreiber:ESP32_Joy-it -> Fernschreiber:IC-Fassung-6pol
- moved J3 94.7 mm to (95.5, 43.5), turned to 90 degrees
- moved J4 85.2 mm to (57.0, 43.5), turned to 90 degrees
- moved D2 78.9 mm to (60.0, 137.5)
- moved J9 70.2 mm to (75.6, 105.0), turned to 0 degrees
- moved J11 67.2 mm to (65.0, 112.1), turned to 0 degrees
- moved D1 63.7 mm to (80.0, 127.0)
- moved J5 63.3 mm to (111.0, 43.5), turned to 90 degrees
- moved J1 54.1 mm to (110.0, 130.0)
- moved J7 52.3 mm to (52.0, 80.1), turned to 270 degrees
- moved J2 48.0 mm to (90.0, 130.0)
- moved R3 44.0 mm to (54.0, 126.7), turned to 270 degrees
- moved R9 41.6 mm to (69.8, 92.0), turned to 0 degrees
- moved Q2 41.3 mm to (64.0, 88.5), turned to 180 degrees
- moved U3 40.5 mm to (68.5, 105.0), turned to 270 degrees
- moved J6 38.4 mm to (130.0, 130.0)
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Connections:
- D1 pad 1: Net-(5V1-Pad3) -> /5V
- D1 pad 2: Net-(D1-Pad2) -> /Relai_ground
- D2 pad 1: Net-(D1-Pad2) -> /Teleprinter_output
- D3 pad 1: Net-(D3-Pad1) -> /Relai_ground
- J10 pad 1: /3V3 -> /write
- J11 pad 1: /3V3 -> Net-(J11-Pad1)
- J2 pad 2: Net-(5V1-Pad3) -> /Step-up_input
- J3 pad 1: Net-(J3-Pad1) -> /3V3
- J3 pad 2: Net-(J3-Pad2) -> GND
- J4 pad 1: Net-(J4-Pad1) -> /3V3
- J5 pad 1: Net-(J5-Pad1) -> /3V3
- J6 pad 2: Net-(C3-Pad1) -> /5V
- J7 pad 1: GND -> /3V3
- J7 pad 2: /3V3 -> GND
- J8 pad 1: Net-(J8-Pad1) -> /Voltage_reversal_Relai
- J9 pad 1: +12V -> /read
- K1 pad 11: Net-(J3-Pad1) -> Net-(J1-Pad1)
- K1 pad 12: Net-(C3-Pad1) -> /Step-up_input
- K1 pad 14: Net-(D3-Pad1) -> /Teleprinter_output
- K1 pad A1: Net-(D1-Pad2) -> /Relai_ground
- K1 pad A2: Net-(5V1-Pad3) -> /5V
- K2 pad 11: Net-(J3-Pad2) -> Net-(J1-Pad2)
- K2 pad 12: Net-(D3-Pad1) -> /Teleprinter_output
- K2 pad 14: Net-(C3-Pad1) -> /Step-up_input
- K2 pad A1: Net-(D1-Pad2) -> /Relai_ground
- K2 pad A2: Net-(5V1-Pad3) -> /5V
- Q1 pad 3: Net-(D1-Pad2) -> /Relai_ground
- Q2 pad 2: Net-(J4-Pad1) -> /write
- R1 pad 1: /Spannungsumkehr_Relai -> /Voltage_reversal_Relai
- R1 pad 2: Net-(J1-Pad1) -> Net-(R1-Pad2)
- R2 pad 1: Net-(5V1-Pad3) -> /5V
- R3 pad 1: Net-(J4-Pad1) -> /Teleprinter_output
- R3 pad 2: GND -> Net-(R3-Pad2)
- R4 pad 1: Net-(D3-Pad1) -> Net-(R3-Pad2)
- R6 pad 2: Net-(R6-Pad2) -> Net-(Q2-Pad3)
- R7 pad 1: Net-(R6-Pad2) -> /write
- R7 pad 2: Net-(Q2-Pad3) -> GND
- R8 pad 1: Net-(D3-Pad1) -> /Teleprinter_output
- R8 pad 2: Net-(J5-Pad1) -> Net-(J11-Pad1)
- R9 pad 1: /3V3 -> /read
- R9 pad 2: Net-(J8-Pad1) -> /3V3
- U1 pad 1: Net-(J1-Pad1) -> Net-(R1-Pad2)
- U2 pad 1: Net-(J5-Pad1) -> /D23
- U2 pad 2: GND -> (no net)
- U2 pad 3: (no net) -> /TX0
- U2 pad 4: GND -> /RX0
- U2 pad 5: Net-(J8-Pad1) -> (no net)
- U2 pad 6: (no net) -> /D19
- U3 pad 1: /D23 -> Net-(J11-Pad1)
- U3 pad 2: (no net) -> Net-(Q2-Pad3)
- U3 pad 3: /TX0 -> (no net)
- U3 pad 4: /RX0 -> GND
- U3 pad 5: (no net) -> /read
- U3 pad 6: /D19 -> (no net)
Routing:
- net /5V: track 0.00 -> 206.6 mm
- net Net-(D3-Pad1): track 100.1 -> 0.00 mm
- net /Teleprinter_output: track 0.00 -> 95.8 mm
- net Net-(5V1-Pad3): track 86.7 -> 0.00 mm
- net Net-(C3-Pad1): track 82.7 -> 0.00 mm
- net Net-(D1-Pad2): track 82.5 -> 0.00 mm
- net GND: track 77.0 -> 0.02 mm
- net /Relai_ground: track 0.00 -> 64.3 mm
- net Net-(J4-Pad1): track 62.5 -> 0.00 mm
- net /3V3: track 196.2 -> 140.7 mm
- net Net-(J8-Pad1): track 54.1 -> 0.00 mm
- net /Step-up_input: track 0.00 -> 46.3 mm
- net Net-(J1-Pad2): track 0.00 -> 44.0 mm
- net +12V: track 43.5 -> 0.00 mm
- net /read: track 0.00 -> 32.8 mm
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Other:
- board text added: "+"
- board text added: "-"
- board text added: "3V3"
- board text added: "3V3>"
- board text added: "5V"
- board text added: "60V"
- board text added: ">"
- board text added: "D18>"
- board text added: "D19>"
- board text added: "D23>"
- board text added: "GND"
- board text added: "GND>"
- board text added: "RX0>"
- board text added: "TX0>"
- board text added: "Teleprinter-FSG Rev. 2 Design by Metzler Benedikt"
- board text removed: "Power 12V"
- board text removed: "Step-Up 60V"
- board text removed: "Teleprinter-FSG Rev. 1 Design by Metzler Benedikt"

Commit message: Updated PCB
Parts:
- added C1: CAP, Capacitor_THT:CP_Radial_D8.0mm_P3.50mm, F.Cu at (106.5, 103.0)
- added C2: CAP, Capacitor_THT:CP_Radial_D8.0mm_P3.50mm, F.Cu at (96.5, 103.0)
- added C3: CAP, Capacitor_THT:CP_Radial_D8.0mm_P3.50mm, F.Cu at (106.5, 97.0)
- added G***: LOGO, Fernschreiber:HTR_Logo, F.Cu at (66.0, 62.9)
- added G***: LOGO, Fernschreiber:Signatur, F.Cu at (128.2, 46.7)
- added H1: MountingHole_Pad, Fernschreiber:Hole, F.Cu at (49.0, 44.5)
- added H2: MountingHole_Pad, Fernschreiber:Hole, F.Cu at (142.2, 44.5)
- added H3: MountingHole_Pad, Fernschreiber:Hole, F.Cu at (49.0, 137.8)
- added H4: MountingHole_Pad, Fernschreiber:Hole, F.Cu at (142.2, 137.8)
- added J12: Conn_01x05_Male, Fernschreiber:stepdown, F.Cu at (127.0, 76.0)
- moved J10 0.30 mm to (72.2, 82.4)
- moved J8 0.14 mm to (64.4, 98.0)
Connections:
- J6 pad 2: /5V -> /5V_12V
Routing:
- net /5V_12V: track 0.00 -> 32.1 mm
- net /5V: track 206.6 -> 222.1 mm
- net Net-(Q1-Pad2): track 32.8 -> 30.9 mm
- net /Teleprinter_output: track 95.8 -> 97.3 mm
- net /Step-up_input: track 46.3 -> 47.8 mm
- net /3V3: track 140.7 -> 139.8 mm
- net Net-(J1-Pad1): track 28.9 -> 29.7 mm
- net Net-(Q2-Pad3): track 18.5 -> 19.2 mm
- net GND: vias 0 -> 2
Other:
- board text added: "5V (12V)"
- board text added: "ABBA"
- board text added: "J1: Teleprinter J2: Stepup 60V J3: 3V3 GND D18 D19 D23 J4: 3V3 GND D13 D12 D14 J5: 3V3 GND RX0 TX0 J6: 5V (12V) J7: Testcon GND 3V3 J8: Testcon Relay Controll (3V3) J9: Testcon READ (3V3) J10: Testcon WRITE (3V3) J11: Testcon OPTO from TelePrinter J12: Stepdown 5V"
- board text removed: "J1 : Relay Controll J2 : GND 5V J3 : Teleprinter Connetion J4 : Write J5 : Read befor Opto J6 : Step-Up 60V J7 : GND 3V3 J8 : Read after Opto J9 : Supply 12V J10: 3V3 GND D18 D19 D23 J11: 3V3 GND D12 D13 D14 J12: 3V3 GND RX0 TX0"
